Commit message: Almost achieved peg-based control, still working out correct TF tree functions.

File: urdf/robotiq_gripper.xacro (robot description, xacro)
@@ -46,4 +46,6 @@
       </collision>
     </link>
+    <link name="${parent}_to_gripper_tip_link">
+    </link>
     <joint name="${parent}tool0_to_eoat_link" type="fixed">
         <parent link="${parent}" />
@@ -51,4 +53,9 @@
         <origin rpy="0.0 0.0 0" xyz="0.00 0.00 0.00" />
     </joint>
+    <joint name="${parent}_gripper_TCP_joint" type="fixed">
+        <parent link="tool0" />
+        <child link="${parent}_to_gripper_tip_link" />
+        <origin rpy="0.0 0.0 0" xyz="0.00 0.00 0.1700" />
+    </joint>
   </xacro:macro>
 </robot>

Commit message: Reinterpret works now; very low torques are reported for both corner and tip positions. Problem was incorrect tool0_to_gripper_tip_link length; may have been geometrically accurate but did not produce good mathematical results. New value may render in incorrect place on RViz or cause later TCP pose errors; consider workarounds.

File: urdf/robotiq_gripper.xacro (robot description, xacro)
@@ -56,5 +56,5 @@
         <parent link="tool0" />
         <child link="${parent}_to_gripper_tip_link" />
-        <origin rpy="0.0 0.0 0" xyz="0.00 0.00 0.1700" />
+        <origin rpy="0.0 0.0 0" xyz="0.00 0.00 0.0750" />
     </joint>
   </xacro:macro>

Commit message: Added a static offset to wrench reinterpretation to account for distance between load cell and tool0; modified robotiq_gripper.xacro and peg_in_hole_params to reflect real dimensions of robot and peg; tested and working on both corner_search and spiral_search, and works with longer pegs (worked with a pencil).

File: urdf/robotiq_gripper.xacro (robot description, xacro)
@@ -31,5 +31,5 @@
           <cylinder radius="0.015" length="0.175"/>
         </geometry>
-        <origin rpy="0 0 0" xyz="0 0 0.0875" />
+        <origin rpy="0 0 0" xyz="0 0 0.0575" />
         <material name="">
           <color rgba="0.1 0.1 0.1 1" />
@@ -38,7 +38,7 @@
       <collision>
         <geometry>
-          <cylinder radius="0.015" length="0.175"/>
+          <cylinder radius="0.015" length="0.155"/>
         </geometry>
-        <origin rpy="0 0 0" xyz="0 0 0.0875" />
+        <origin rpy="0 0 0" xyz="0 0 0.0575" />
         <material name="">
           <color rgba="0.1 0.1 0.1 1" />
@@ -56,5 +56,5 @@
         <parent link="tool0" />
         <child link="${parent}_to_gripper_tip_link" />
-        <origin rpy="0.0 0.0 0" xyz="0.00 0.00 0.0750" />
+        <origin rpy="0.0 0.0 0" xyz="0.00 0.00 0.115" />
     </joint>
   </xacro:macro>
